Commit message: make .urdf

File: planner/arm_description/urdf/arm.xacro (robot description, xacro)
@@ -1,6 +1,6 @@
 <?xml version="1.0" ?>
 <robot name="arm" xmlns:xacro="http://www.ros.org/wiki/xacro">
-<xacro:include filename="$(find arm_description)/urdf/materials.xacro" />
-<xacro:include filename="$(find arm_description)/urdf/arm.trans" />
+<xacro:include filename="materials.xacro" />
+<xacro:include filename="arm.trans" />
 <link name="base_link">
   <inertial>
@@ -12,5 +12,5 @@
     <origin xyz="0 0 0" rpy="0 0 0"/>
     <geometry>
-      <mesh filename="package://arm_description/meshes/base_link.stl" scale="0.001 0.001 0.001"/>
+      <mesh filename="../meshes/base_link.stl" scale="0.001 0.001 0.001"/>
     </geometry>
     <material name="steel_satin"/>
@@ -19,5 +19,5 @@
     <origin xyz="0 0 0" rpy="0 0 0"/>
     <geometry>
-      <mesh filename="package://arm_description/meshes/base_link.stl" scale="0.001 0.001 0.001"/>
+      <mesh filename="../meshes/base_link.stl" scale="0.001 0.001 0.001"/>
     </geometry>
   </collision>
@@ -32,5 +32,5 @@
     <origin xyz="0.01 0.0005 0.077" rpy="0 0 0"/>
     <geometry>
-      <mesh filename="package://arm_description/meshes/glid_platta_1.stl" scale="0.001 0.001 0.001"/>
+      <mesh filename="../meshes/glid_platta_1.stl" scale="0.001 0.001 0.001"/>
     </geometry>
     <material name="abs_white"/>
@@ -39,5 +39,5 @@
     <origin xyz="0.01 0.0005 0.077" rpy="0 0 0"/>
     <geometry>
-      <mesh filename="package://arm_description/meshes/glid_platta_1.stl" scale="0.001 0.001 0.001"/>
+      <mesh filename="../meshes/glid_platta_1.stl" scale="0.001 0.001 0.001"/>
     </geometry>
   </collision>
@@ -52,5 +52,5 @@
     <origin xyz="0.04 0.0955 0.061" rpy="0 0 0"/>
     <geometry>
-      <mesh filename="package://arm_description/meshes/bas_1.stl" scale="0.001 0.001 0.001"/>
+      <mesh filename="../meshes/bas_1.stl" scale="0.001 0.001 0.001"/>
     </geometry>
     <material name="abs_white"/>
@@ -59,5 +59,5 @@
     <origin xyz="0.04 0.0955 0.061" rpy="0 0 0"/>
     <geometry>
-      <mesh filename="package://arm_description/meshes/bas_1.stl" scale="0.001 0.001 0.001"/>
+      <mesh filename="../meshes/bas_1.stl" scale="0.001 0.001 0.001"/>
     </geometry>
   </collision>
@@ -72,5 +72,5 @@
     <origin xyz="0.025 0.006 0.0565" rpy="0 0 0"/>
     <geometry>
-      <mesh filename="package://arm_description/meshes/gemensam_vagg_1.stl" scale="0.001 0.001 0.001"/>
+      <mesh filename="../meshes/gemensam_vagg_1.stl" scale="0.001 0.001 0.001"/>
     </geometry>
     <material name="abs_white"/>
@@ -79,5 +79,5 @@
     <origin xyz="0.025 0.006 0.0565" rpy="0 0 0"/>
     <geometry>
-      <mesh filename="package://arm_description/meshes/gemensam_vagg_1.stl" scale="0.001 0.001 0.001"/>
+      <mesh filename="../meshes/gemensam_vagg_1.stl" scale="0.001 0.001 0.001"/>
     </geometry>
   </collision>
@@ -92,5 +92,5 @@
     <origin xyz="0.0175 0.0083 0.016" rpy="0 0 0"/>
     <geometry>
-      <mesh filename="package://arm_description/meshes/botten_snurr_1.stl" scale="0.001 0.001 0.001"/>
+      <mesh filename="../meshes/botten_snurr_1.stl" scale="0.001 0.001 0.001"/>
     </geometry>
     <material name="abs_white"/>
@@ -99,5 +99,5 @@
     <origin xyz="0.0175 0.0083 0.016" rpy="0 0 0"/>
     <geometry>
-      <mesh filename="package://arm_description/meshes/botten_snurr_1.stl" scale="0.001 0.001 0.001"/>
+      <mesh filename="../meshes/botten_snurr_1.stl" scale="0.001 0.001 0.001"/>
     </geometry>
   </collision>
@@ -112,5 +112,5 @@
     <origin xyz="0.0265 0.0173 0.001" rpy="0 0 0"/>
     <geometry>
-      <mesh filename="package://arm_description/meshes/kortarm_kopia_Mirror__1.stl" scale="0.001 0.001 0.001"/>
+      <mesh filename="../meshes/kortarm_kopia_Mirror__1.stl" scale="0.001 0.001 0.001"/>
     </geometry>
     <material name="abs_white"/>
@@ -119,5 +119,5 @@
     <origin xyz="0.0265 0.0173 0.001" rpy="0 0 0"/>
     <geometry>
-      <mesh filename="package://arm_description/meshes/kortarm_kopia_Mirror__1.stl" scale="0.001 0.001 0.001"/>
+      <mesh filename="../meshes/kortarm_kopia_Mirror__1.stl" scale="0.001 0.001 0.001"/>
     </geometry>
   </collision>
@@ -132,5 +132,5 @@
     <origin xyz="0.0085 0.0673 0.001" rpy="0 0 0"/>
     <geometry>
-      <mesh filename="package://arm_description/meshes/kortarm_kopia_1.stl" scale="0.001 0.001 0.001"/>
+      <mesh filename="../meshes/kortarm_kopia_1.stl" scale="0.001 0.001 0.001"/>
     </geometry>
     <material name="abs_white"/>
@@ -139,5 +139,5 @@
     <origin xyz="0.0085 0.0673 0.001" rpy="0 0 0"/>
     <geometry>
-      <mesh filename="package://arm_description/meshes/kortarm_kopia_1.stl" scale="0.001 0.001 0.001"/>
+      <mesh filename="../meshes/kortarm_kopia_1.stl" scale="0.001 0.001 0.001"/>
     </geometry>
   </collision>
@@ -152,5 +152,5 @@
     <origin xyz="0.01 0.08 0.0565" rpy="0 0 0"/>
     <geometry>
-      <mesh filename="package://arm_description/meshes/snurr_hallare_stepper_sida_1.stl" scale="0.001 0.001 0.001"/>
+      <mesh filename="../meshes/snurr_hallare_stepper_sida_1.stl" scale="0.001 0.001 0.001"/>
     </geometry>
     <material name="acetal_resin_white"/>
@@ -159,5 +159,5 @@
     <origin xyz="0.01 0.08 0.0565" rpy="0 0 0"/>
     <geometry>
-      <mesh filename="package://arm_description/meshes/snurr_hallare_stepper_sida_1.stl" scale="0.001 0.001 0.001"/>
+      <mesh filename="../meshes/snurr_hallare_stepper_sida_1.stl" scale="0.001 0.001 0.001"/>
     </geometry>
   </collision>
@@ -172,5 +172,5 @@
     <origin xyz="0.025 0.0633 -0.244" rpy="0 0 0"/>
     <geometry>
-      <mesh filename="package://arm_description/meshes/led_1.stl" scale="0.001 0.001 0.001"/>
+      <mesh filename="../meshes/led_1.stl" scale="0.001 0.001 0.001"/>
     </geometry>
     <material name="abs_white"/>
@@ -179,5 +179,5 @@
     <origin xyz="0.025 0.0633 -0.244" rpy="0 0 0"/>
     <geometry>
-      <mesh filename="package://arm_description/meshes/led_1.stl" scale="0.001 0.001 0.001"/>
+      <mesh filename="../meshes/led_1.stl" scale="0.001 0.001 0.001"/>
     </geometry>
   </collision>
@@ -192,5 +192,5 @@
     <origin xyz="0.3074 0.0167 -0.273879" rpy="0 0 0"/>
     <geometry>
-      <mesh filename="package://arm_description/meshes/mount_1.stl" scale="0.001 0.001 0.001"/>
+      <mesh filename="../meshes/mount_1.stl" scale="0.001 0.001 0.001"/>
     </geometry>
     <material name="abs_white"/>
@@ -199,5 +199,5 @@
     <origin xyz="0.3074 0.0167 -0.273879" rpy="0 0 0"/>
     <geometry>
-      <mesh filename="package://arm_description/meshes/mount_1.stl" scale="0.001 0.001 0.001"/>
+      <mesh filename="../meshes/mount_1.stl" scale="0.001 0.001 0.001"/>
     </geometry>
   </collision>
@@ -212,5 +212,5 @@
     <origin xyz="0.0175 0.0257 -0.274" rpy="0 0 0"/>
     <geometry>
-      <mesh filename="package://arm_description/meshes/led_axel_1.stl" scale="0.001 0.001 0.001"/>
+      <mesh filename="../meshes/led_axel_1.stl" scale="0.001 0.001 0.001"/>
     </geometry>
     <material name="abs_white"/>
@@ -219,5 +219,5 @@
     <origin xyz="0.0175 0.0257 -0.274" rpy="0 0 0"/>
     <geometry>
-      <mesh filename="package://arm_description/meshes/led_axel_1.stl" scale="0.001 0.001 0.001"/>
+      <mesh filename="../meshes/led_axel_1.stl" scale="0.001 0.001 0.001"/>
     </geometry>
   </collision>
@@ -232,5 +232,5 @@
     <origin xyz="0.019 0.0127 -0.277708" rpy="0 0 0"/>
     <geometry>
-      <mesh filename="package://arm_description/meshes/lang_arm_1.stl" scale="0.001 0.001 0.001"/>
+      <mesh filename="../meshes/lang_arm_1.stl" scale="0.001 0.001 0.001"/>
     </geometry>
     <material name="abs_white"/>
@@ -239,5 +239,5 @@
     <origin xyz="0.019 0.0127 -0.277708" rpy="0 0 0"/>
     <geometry>
-      <mesh filename="package://arm_description/meshes/lang_arm_1.stl" scale="0.001 0.001 0.001"/>
+      <mesh filename="../meshes/lang_arm_1.stl" scale="0.001 0.001 0.001"/>
     </geometry>
   </collision>
@@ -252,5 +252,5 @@
     <origin xyz="0.019 0.0727 -0.277708" rpy="0 0 0"/>
     <geometry>
-      <mesh filename="package://arm_description/meshes/lang_arm_Mirror__1.stl" scale="0.001 0.001 0.001"/>
+      <mesh filename="../meshes/lang_arm_Mirror__1.stl" scale="0.001 0.001 0.001"/>
     </geometry>
     <material name="abs_white"/>
@@ -259,5 +259,5 @@
     <origin xyz="0.019 0.0727 -0.277708" rpy="0 0 0"/>
     <geometry>
-      <mesh filename="package://arm_description/meshes/lang_arm_Mirror__1.stl" scale="0.001 0.001 0.001"/>
+      <mesh filename="../meshes/lang_arm_Mirror__1.stl" scale="0.001 0.001 0.001"/>
     </geometry>
   </collision>
@@ -272,5 +272,5 @@
     <origin xyz="0.3114 0.0517 -0.283879" rpy="0 0 0"/>
     <geometry>
-      <mesh filename="package://arm_description/meshes/ram_1.stl" scale="0.001 0.001 0.001"/>
+      <mesh filename="../meshes/ram_1.stl" scale="0.001 0.001 0.001"/>
     </geometry>
     <material name="abs_white"/>
@@ -279,5 +279,5 @@
     <origin xyz="0.3114 0.0517 -0.283879" rpy="0 0 0"/>
     <geometry>
-      <mesh filename="package://arm_description/meshes/ram_1.stl" scale="0.001 0.001 0.001"/>
+      <mesh filename="../meshes/ram_1.stl" scale="0.001 0.001 0.001"/>
     </geometry>
   </collision>
@@ -292,5 +292,5 @@
     <origin xyz="0.029306 0.0026 -0.005" rpy="0 0 0"/>
     <geometry>
-      <mesh filename="package://arm_description/meshes/Component18_1.stl" scale="0.001 0.001 0.001"/>
+      <mesh filename="../meshes/Component18_1.stl" scale="0.001 0.001 0.001"/>
     </geometry>
     <material name="abs_white"/>
@@ -299,5 +299,5 @@
     <origin xyz="0.029306 0.0026 -0.005" rpy="0 0 0"/>
     <geometry>
-      <mesh filename="package://arm_description/meshes/Component18_1.stl" scale="0.001 0.001 0.001"/>
+      <mesh filename="../meshes/Component18_1.stl" scale="0.001 0.001 0.001"/>
     </geometry>
   </collision>
@@ -312,5 +312,5 @@
     <origin xyz="0.3333 0.015006 -0.261879" rpy="0 0 0"/>
     <geometry>
-      <mesh filename="package://arm_description/meshes/hake_1.stl" scale="0.001 0.001 0.001"/>
+      <mesh filename="../meshes/hake_1.stl" scale="0.001 0.001 0.001"/>
     </geometry>
     <material name="abs_white"/>
@@ -319,5 +319,5 @@
     <origin xyz="0.3333 0.015006 -0.261879" rpy="0 0 0"/>
     <geometry>
-      <mesh filename="package://arm_description/meshes/hake_1.stl" scale="0.001 0.001 0.001"/>
+      <mesh filename="../meshes/hake_1.stl" scale="0.001 0.001 0.001"/>
     </geometry>
   </collision>
@@ -332,5 +332,5 @@
     <origin xyz="0.3383 0.073006 -0.261879" rpy="0 0 0"/>
     <geometry>
-      <mesh filename="package://arm_description/meshes/hake2_1.stl" scale="0.001 0.001 0.001"/>
+      <mesh filename="../meshes/hake2_1.stl" scale="0.001 0.001 0.001"/>
     </geometry>
     <material name="abs_white"/>
@@ -339,5 +339,5 @@
     <origin xyz="0.3383 0.073006 -0.261879" rpy="0 0 0"/>
     <geometry>
-      <mesh filename="package://arm_description/meshes/hake2_1.stl" scale="0.001 0.001 0.001"/>
+      <mesh filename="../meshes/hake2_1.stl" scale="0.001 0.001 0.001"/>
     </geometry>
   </collision>
